File: project/ngff.sch (KiCad schematic (older format))
At the start: 55 parts, among them J1 KUSBX-BS1N9-1-BL30, J2 2199119-3, J3 Jack-DC, J4 SIM8060-6-1-14-00-A, J5 Conn_01x03_Male, J6 SIM8060-6-1-14-00-A, SW1 KMR221GLFS, U1 AP62301WU7

Commit message: update
Parts:
- U1: symbol Power_Management:AP62301WU7 -> ngff-rescue:AP62301WU7-Power_Management
Changed lines of the file:
@@
 $EndComp
 $Comp
-L Power_Management:AP62301WU7 U1
+L ngff-rescue:AP62301WU7-Power_Management U1
 U 1 1 609318E9
 P 3350 6650
